File: KiCad/AQM AGS10.kicad_pcb (KiCad board)
At the start: 2 copper layers, 99.8 x 50 mm, 26 parts, among them U2 XIAO-RP2040-SMD, U3 MCP73831T-2ACI_OT

Commit message: Add files via upload
Parts:
- D2: footprint Diode_SMD:D_0603_1608Metric -> Diode_SMD:D_SOD-123
- moved R1 26.7 mm to (122.0, 93.3)
- moved U1 23.7 mm to (123.3, 96.8), turned to -90 degrees
- moved C1 23.5 mm to (122.8, 99.8), turned to 0 degrees
- moved R2 20.8 mm to (124.6, 93.3), turned to 180 degrees
- moved R5 2.76 mm to (151.1, 72.2)
Connections:
- U1 pad 1: (no net) -> /SCL
- U1 pad 2: (no net) -> /SDA
- U1 pad 3: (no net) -> GND
- U1 pad 4: (no net) -> +3V3
Routing:
- net /SDA: track 38.9 -> 20.0 mm
- net /SCL: track 35.4 -> 17.7 mm
- net Net-(U2-GPIO29_A3_D3): track 42.4 -> 38.7 mm
- net GND: track 15.1 -> 18.4 mm, vias 1 -> 2
- net /BAT: track 39.3 -> 40.8 mm
- net +3V3: track 60.9 -> 59.7 mm
- net +5V: track 47.8 -> 47.1 mm
