File: KiCad/AQM AGS10.kicad_sch (KiCad schematic)
At the start: 26 parts, among them U2 XIAO-RP2040-SMD, U3 MCP73831T-2ACI_OT

Commit message: Add files via upload
Parts:
- D2: footprint Diode_SMD:D_0603_1608Metric -> Diode_SMD:D_SOD-123
Changed lines of the file:
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@@
 			)
 		)
-		(property "Footprint" "Diode_SMD:D_0603_1608Metric"
+		(property "Footprint" "Diode_SMD:D_SOD-123"
 			(at 191.77 77.47 90)
 			(hide yes)
